Commit message: feat: add laser scanner

File: urdf/wheel_bot.xacro (robot description, xacro)
@@ -136,4 +136,12 @@
     <joint_properties damping="1.0" friction="1.0"/>
   </joint>
+  <joint type="fixed" name="camera_joint">
+    <origin xyz="0.2 0 0" rpy="0 0 0"/>
+    <child link="camera"/>
+    <parent link="chassis"/>
+    <axis xyz="0 1 0" rpy="0 0 0"/>
+    <limit effort="10000" velocity="1000"/>
+    <joint_properties damping="1.0" friction="1.0"/>
+  </joint>
   <link name='camera'>
     <inertial>
@@ -158,11 +166,35 @@
     </visual>
   </link>
-  <joint type="fixed" name="camera_joint">
-    <origin xyz="0.2 0 0" rpy="0 0 0"/>
-    <child link="camera"/>
-    <parent link="chassis"/>
-    <axis xyz="0 1 0" rpy="0 0 0"/>
-    <limit effort="10000" velocity="1000"/>
-    <joint_properties damping="1.0" friction="1.0"/>
-  </joint>
+  <!-- laser scanner -->
+  <joint type="fixed" name="hokuyo_joint">
+    <origin xyz="0.15 0 0.1" rpy="0 0 0"/>
+    <child link="hokuyo"/>
+    <parent link="chassis"/>
+    <axis xyz="0 1 0" rpy="0 0 0"/>
+    <limit effort="10000" velocity="1000"/>
+    <joint_properties damping="1.0" friction="1.0"/>
+  </joint>
+  <link name='hokuyo'>
+    <pose>0 0 0 0 0 0</pose>
+    <inertial>
+      <mass value="0.1"/>
+      <origin xyz="0 0 0" rpy=" 0 0 0"/>
+      <inertia
+          ixx="1e-6" ixy="0" ixz="0"
+          iyy="1e-6" iyz="0"
+          izz="1e-6" />
+    </inertial>
+    <collision name='hokuyo_collision'>
+      <origin xyz="0 0 0" rpy=" 0 0 0"/>
+      <geometry>
+        <box size=".1 .1 .1"/>
+      </geometry>
+    </collision>
+    <visual name='hokuyo_visual'>
+      <origin xyz="0 0 0" rpy=" 0 0 0"/>
+      <geometry>
+        <mesh filename="package://udacity_bot/meshes/hokuyo.dae"/>
+      </geometry>
+    </visual>
+  </link>
 </robot>

Commit message: feat: add kinect model

File: urdf/wheel_bot.xacro (robot description, xacro)
@@ -136,13 +136,14 @@
     <joint_properties damping="1.0" friction="1.0"/>
   </joint>
+  <!-- RGB-D camera Kinect -->
   <joint type="fixed" name="camera_joint">
-    <origin xyz="0.2 0 0" rpy="0 0 0"/>
-    <child link="camera"/>
-    <parent link="chassis"/>
-    <axis xyz="0 1 0" rpy="0 0 0"/>
-    <limit effort="10000" velocity="1000"/>
-    <joint_properties damping="1.0" friction="1.0"/>
-  </joint>
-  <link name='camera'>
+    <origin xyz="0.2 0 0.1" rpy="0 0 0"/>
+    <child link="camera_link"/>
+    <parent link="chassis"/>
+    <axis xyz="0 1 0" rpy="0 0 0"/>
+    <limit effort="10000" velocity="1000"/>
+    <joint_properties damping="1.0" friction="1.0"/>
+  </joint>
+  <link name='camera_link'>
     <inertial>
       <mass value="0.1"/>
@@ -156,5 +157,5 @@
       <origin xyz="0 0 0" rpy=" 0 0 0"/>
       <geometry>
-        <box size=".05 .05 .05"/>
+        <box size=".05 .22 .1"/>
       </geometry>
     </collision>
@@ -162,5 +163,5 @@
       <origin xyz="0 0 0" rpy=" 0 0 0"/>
       <geometry>
-        <box size=".05 .05 .05"/>
+        <mesh filename="package://rtab_slam/meshes/kinect.dae"/>
       </geometry>
     </visual>
@@ -168,5 +169,5 @@
   <!-- laser scanner -->
   <joint type="fixed" name="hokuyo_joint">
-    <origin xyz="0.15 0 0.1" rpy="0 0 0"/>
+    <origin xyz="0.1 0 0.125" rpy="0 0 0"/>
     <child link="hokuyo"/>
     <parent link="chassis"/>
@@ -194,5 +195,5 @@
       <origin xyz="0 0 0" rpy=" 0 0 0"/>
       <geometry>
-        <mesh filename="package://udacity_bot/meshes/hokuyo.dae"/>
+        <mesh filename="package://rtab_slam/meshes/hokuyo.dae"/>
       </geometry>
     </visual>

Commit message: feat: add kinect with pointcloud transform

File: urdf/wheel_bot.xacro (robot description, xacro)
@@ -2,4 +2,5 @@
 <robot name="rtab_slam" xmlns:xacro="http://www.ros.org/wiki/xacro">
   <xacro:include filename="$(find rtab_slam)/urdf/wheel_bot.gazebo" />
+  <xacro:property name="M_PI" value="3.14159" />
   <link name="robot_footprint"></link>
   <joint name="robot_footprint_joint" type="fixed">
@@ -167,7 +168,18 @@
     </visual>
   </link>
+  <!-- depth cloud transform for RViz
+      Code modified from sealguy77 from ROS answers
+      https://answers.ros.org/question/206823/kinect-frame/ -->
+  <joint name="kinect_depth_optical_joint" type="fixed">
+    <origin xyz="0 0 0" rpy="${-M_PI/2} 0 ${-M_PI/2}" />
+    <parent link="camera_link" />
+    <child link="kinect_depth_optical_frame" />
+  </joint>
+  <!-- link to this frame to transform the point cloud -->
+  <!-- <frameName>kinect_depth_optical_frame</frameName> -->
+  <link name="kinect_depth_optical_frame" />
   <!-- laser scanner -->
   <joint type="fixed" name="hokuyo_joint">
-    <origin xyz="0.1 0 0.125" rpy="0 0 0"/>
+    <origin xyz="0.1 0 0.15" rpy="0 0 0"/>
     <child link="hokuyo"/>
     <parent link="chassis"/>

Commit message: chore: fix laser and kinect collision box

File: urdf/wheel_bot.xacro (robot description, xacro)
@@ -156,7 +156,7 @@
     </inertial>
     <collision name='camera_collision'>
-      <origin xyz="0 0 0" rpy=" 0 0 0"/>
-      <geometry>
-        <box size=".05 .22 .1"/>
+      <origin xyz="-0.03 0 -0.015" rpy=" 0 0 0"/>
+      <geometry>
+        <box size="0.06 0.28 0.073" />
       </geometry>
     </collision>
@@ -181,5 +181,5 @@
   <!-- laser scanner -->
   <joint type="fixed" name="hokuyo_joint">
-    <origin xyz="0.1 0 0.15" rpy="0 0 0"/>
+    <origin xyz="0.1 0 0.125" rpy="0 0 0"/>
     <child link="hokuyo"/>
     <parent link="chassis"/>

Commit message: feat: working kinect sensor and topics

File: urdf/wheel_bot.xacro (robot description, xacro)
@@ -1,39 +1,55 @@
-<?xml version='1.0'?>
-<robot name="rtab_slam" xmlns:xacro="http://www.ros.org/wiki/xacro">
-  <xacro:include filename="$(find rtab_slam)/urdf/wheel_bot.gazebo" />
-  <xacro:property name="M_PI" value="3.14159" />
+<?xml version="1.0" ?>
+<robot name="wheel_bot" xmlns:xacro="http://www.ros.org/wiki/xacro">
+  <!-- Define constants -->
+  <xacro:property name="M_PI" value="3.1415926535897931" />
+  <xacro:property name="robot_base_link" value="chassis" />
+  <xacro:property name="caster_back_radius" value="0.0495" />
+  <xacro:property name="caster_front_radius" value="0.05" />
+  <xacro:property name="caster_offset_x" value="0.15" />
+  <xacro:property name="caster_offset_y" value="0.0" />
+  <xacro:property name="caster_offset_z" value="-0.05" />
+  <xacro:property name="base_length" value="0.4" />
+  <xacro:property name="base_width" value="0.2" />
+  <xacro:property name="base_height" value="0.1" />
+  <xacro:property name="base_mass" value="15.0" />
+  <xacro:property name="base_ixx" value="${base_mass * (base_width*base_width + base_height*base_height) / 12.0}" />
+  <xacro:property name="base_iyy" value="${base_mass * (base_length*base_length + base_height*base_height) / 12.0}" />
+  <xacro:property name="base_izz" value="${base_mass * (base_length*base_length + base_width*base_height) / 12.0}" />
+  <xacro:include filename="$(find slam_project)/urdf/wheel_bot.gazebo" />
+  <xacro:include filename="$(find slam_project)/urdf/sensor.xacro" />
+  <xacro:include filename="$(find slam_project)/urdf/wheels.xacro" />
+  <!--Links-->
   <link name="robot_footprint"></link>
   <joint name="robot_footprint_joint" type="fixed">
     <origin xyz="0 0 0" rpy="0 0 0" />
     <parent link="robot_footprint"/>
-    <child link="chassis" />
+    <child link="${robot_base_link}" />
   </joint>
-  <link name='chassis'>
+  <link name='${robot_base_link}'>
     <pose>0 0 0.1 0 0 0</pose>
     <inertial>
-      <mass value="15.0"/>
-      <origin xyz="0.0 0 0" rpy=" 0 0 0"/>
+      <mass value="${base_mass}"/>
+      <origin xyz="0 0 0" rpy=" 0 0 0"/>
       <inertia
-          ixx="0.1" ixy="0" ixz="0"
-          iyy="0.1" iyz="0"
-          izz="0.1"
-      />
-    </inertial>
-    <collision name='collision'>
+        ixx="${base_ixx}" ixy="0" ixz="0"
+        iyy="${base_iyy}" iyz="0"
+        izz="${base_izz}" />
+      </inertial>
+    <collision>
       <origin xyz="0 0 0" rpy=" 0 0 0"/>
       <geometry>
-        <box size=".4 .2 .1"/>
+        <box size="${base_length} ${base_width} ${base_height}"/>
       </geometry>
     </collision>
-    <visual name='chassis_visual'>
+    <visual>
       <origin xyz="0 0 0" rpy=" 0 0 0"/>
       <geometry>
-        <box size=".4 .2 .1"/>
+        <box size="${base_length} ${base_width} ${base_height}"/>
       </geometry>
     </visual>
     <collision name='back_caster_collision'>
-      <origin xyz="-0.15 0 -0.05" rpy=" 0 0 0"/>
+      <origin xyz="${-caster_offset_x} ${caster_offset_y} ${caster_offset_z}" rpy=" 0 0 0"/>
       <geometry>
-        <sphere radius="0.0495"/>
+        <sphere radius="${caster_back_radius}"/>
       </geometry>
       <surface>
@@ -49,13 +65,13 @@
     </collision>
     <visual name='back_caster_visual'>
-      <origin xyz="-0.15 0 -0.05" rpy=" 0 0 0"/>
+      <origin xyz="${-caster_offset_x} ${caster_offset_y} ${caster_offset_z}" rpy=" 0 0 0"/>
       <geometry>
-        <sphere radius="0.0495"/>
+        <sphere radius="${caster_back_radius}"/>
       </geometry>
     </visual>
     <collision name='front_caster_collision'>
-      <origin xyz="0.15 0 -0.05" rpy=" 0 0 0"/>
+      <origin xyz="${caster_offset_x} ${caster_offset_y} ${caster_offset_z}" rpy=" 0 0 0"/>
       <geometry>
-        <sphere radius="0.05"/>
+        <sphere radius="${caster_front_radius}"/>
       </geometry>
       <surface>
@@ -71,141 +87,7 @@
     </collision>
     <visual name='front_caster_visual'>
-      <origin xyz="0.15 0 -0.05" rpy=" 0 0 0"/>
+      <origin xyz="${caster_offset_x} ${caster_offset_y} ${caster_offset_z}" rpy=" 0 0 0"/>
       <geometry>
-        <sphere radius="0.05"/>
-      </geometry>
-    </visual>
-  </link>
-  <link name="left_wheel">
-    <inertial>
-      <mass value="5.0"/>
-      <origin xyz="0.0 0 0" rpy=" 0 1.5707 1.5707"/>
-      <inertia
-          ixx="0.1" ixy="0" ixz="0"
-          iyy="0.1" iyz="0"
-          izz="0.1" />
-    </inertial>
-    <collision name="left_wheel_collision">
-      <origin xyz="0 0 0" rpy=" 0 1.5707 1.5707"/>
-      <geometry>
-        <cylinder length="0.05" radius="0.1"/>
-      </geometry>
-    </collision>
-    <visual name="left_wheel_visual">
-      <origin xyz="0 0 0" rpy=" 0 1.5707 1.5707"/>
-      <geometry>
-        <cylinder length="0.05" radius="0.1"/>
-      </geometry>
-    </visual>
-  </link>
-  <joint type="continuous" name="left_wheel_hinge">
-    <origin xyz="0 0.15 0" rpy="0 0 0"/>
-    <child link="left_wheel"/>
-    <parent link="chassis"/>
-    <axis xyz="0 1 0" rpy="0 0 0"/>
-    <limit effort="10000" velocity="1000"/>
-    <joint_properties damping="1.0" friction="1.0"/>
-  </joint>
-  <link name="right_wheel">
-    <inertial>
-      <mass value="5.0"/>
-      <origin xyz="0.0 0 0" rpy=" 0 1.5707 1.5707"/>
-      <inertia
-          ixx="0.1" ixy="0" ixz="0"
-          iyy="0.1" iyz="0"
-          izz="0.1" />
-    </inertial>
-    <collision name="right_wheel_collision">
-      <origin xyz="0 0 0" rpy=" 0 1.5707 1.5707"/>
-      <geometry>
-        <cylinder length="0.05" radius="0.1"/>
-      </geometry>
-    </collision>
-    <visual name="right_wheel_visual">
-      <origin xyz="0 0 0" rpy=" 0 1.5707 1.5707"/>
-      <geometry>
-        <cylinder length="0.05" radius="0.1"/>
-      </geometry>
-    </visual>
-  </link>
-  <joint type="continuous" name="right_wheel_hinge">
-    <origin xyz="0 -0.15 0" rpy="0 0 0"/>
-    <child link="right_wheel"/>
-    <parent link="chassis"/>
-    <axis xyz="0 1 0" rpy="0 0 0"/>
-    <limit effort="10000" velocity="1000"/>
-    <joint_properties damping="1.0" friction="1.0"/>
-  </joint>
-  <!-- RGB-D camera Kinect -->
-  <joint type="fixed" name="camera_joint">
-    <origin xyz="0.2 0 0.1" rpy="0 0 0"/>
-    <child link="camera_link"/>
-    <parent link="chassis"/>
-    <axis xyz="0 1 0" rpy="0 0 0"/>
-    <limit effort="10000" velocity="1000"/>
-    <joint_properties damping="1.0" friction="1.0"/>
-  </joint>
-  <link name='camera_link'>
-    <inertial>
-      <mass value="0.1"/>
-      <origin xyz="0.0 0 0" rpy=" 0 0 0"/>
-      <inertia
-          ixx="1e-6" ixy="0" ixz="0"
-          iyy="1e-6" iyz="0"
-          izz="1e-6"/>
-    </inertial>
-    <collision name='camera_collision'>
-      <origin xyz="-0.03 0 -0.015" rpy=" 0 0 0"/>
-      <geometry>
-        <box size="0.06 0.28 0.073" />
-      </geometry>
-    </collision>
-    <visual name='camera_visual'>
-      <origin xyz="0 0 0" rpy=" 0 0 0"/>
-      <geometry>
-        <mesh filename="package://rtab_slam/meshes/kinect.dae"/>
-      </geometry>
-    </visual>
-  </link>
-  <!-- depth cloud transform for RViz
-      Code modified from sealguy77 from ROS answers
-      https://answers.ros.org/question/206823/kinect-frame/ -->
-  <joint name="kinect_depth_optical_joint" type="fixed">
-    <origin xyz="0 0 0" rpy="${-M_PI/2} 0 ${-M_PI/2}" />
-    <parent link="camera_link" />
-    <child link="kinect_depth_optical_frame" />
-  </joint>
-  <!-- link to this frame to transform the point cloud -->
-  <!-- <frameName>kinect_depth_optical_frame</frameName> -->
-  <link name="kinect_depth_optical_frame" />
-  <!-- laser scanner -->
-  <joint type="fixed" name="hokuyo_joint">
-    <origin xyz="0.1 0 0.125" rpy="0 0 0"/>
-    <child link="hokuyo"/>
-    <parent link="chassis"/>
-    <axis xyz="0 1 0" rpy="0 0 0"/>
-    <limit effort="10000" velocity="1000"/>
-    <joint_properties damping="1.0" friction="1.0"/>
-  </joint>
-  <link name='hokuyo'>
-    <pose>0 0 0 0 0 0</pose>
-    <inertial>
-      <mass value="0.1"/>
-      <origin xyz="0 0 0" rpy=" 0 0 0"/>
-      <inertia
-          ixx="1e-6" ixy="0" ixz="0"
-          iyy="1e-6" iyz="0"
-          izz="1e-6" />
-    </inertial>
-    <collision name='hokuyo_collision'>
-      <origin xyz="0 0 0" rpy=" 0 0 0"/>
-      <geometry>
-        <box size=".1 .1 .1"/>
-      </geometry>
-    </collision>
-    <visual name='hokuyo_visual'>
-      <origin xyz="0 0 0" rpy=" 0 0 0"/>
-      <geometry>
-        <mesh filename="package://rtab_slam/meshes/hokuyo.dae"/>
+        <sphere radius="${caster_front_radius}"/>
       </geometry>
     </visual>

Commit message: feat: add SLAM mapping

File: urdf/wheel_bot.xacro (robot description, xacro)
@@ -20,8 +20,8 @@
   <xacro:include filename="$(find slam_project)/urdf/wheels.xacro" />
   <!--Links-->
-  <link name="robot_footprint"></link>
-  <joint name="robot_footprint_joint" type="fixed">
+  <link name="base_footprint"></link>
+  <joint name="base_footprint_joint" type="fixed">
     <origin xyz="0 0 0" rpy="0 0 0" />
-    <parent link="robot_footprint"/>
+    <parent link="base_footprint"/>
     <child link="${robot_base_link}" />
   </joint>

Commit message: chore: update parameters

File: urdf/wheel_bot.xacro (robot description, xacro)
@@ -6,11 +6,11 @@
   <xacro:property name="caster_back_radius" value="0.0495" />
   <xacro:property name="caster_front_radius" value="0.05" />
-  <xacro:property name="caster_offset_x" value="0.15" />
+  <xacro:property name="caster_offset_x" value="${base_length/2 - 0.05}" />
   <xacro:property name="caster_offset_y" value="0.0" />
-  <xacro:property name="caster_offset_z" value="-0.05" />
+  <xacro:property name="caster_offset_z" value="-${caster_front_radius}" />
   <xacro:property name="base_length" value="0.4" />
   <xacro:property name="base_width" value="0.2" />
   <xacro:property name="base_height" value="0.1" />
-  <xacro:property name="base_mass" value="15.0" />
+  <xacro:property name="base_mass" value="20.0" />
   <xacro:property name="base_ixx" value="${base_mass * (base_width*base_width + base_height*base_height) / 12.0}" />
   <xacro:property name="base_iyy" value="${base_mass * (base_length*base_length + base_height*base_height) / 12.0}" />

File: urdf/wheels.xacro (robot description, xacro)
@@ -45,5 +45,5 @@
     </joint>
   </xacro:macro>
-  <xacro:drive_wheel parent="${parent_link}" suffix="left" reflect="1" />
-  <xacro:drive_wheel parent="${parent_link}" suffix="right" reflect="-1" />
+  <xacro:drive_wheel parent="${parent_link}" suffix="left" reflect="-1" />
+  <xacro:drive_wheel parent="${parent_link}" suffix="right" reflect="1" />
 </robot>
